File: design/02_gate_driver.kicad_sch (KiCad schematic)
At the start: 22 parts, among them U201 DRV8323RS

Commit message: PCB floorplan: 80x68 mm, 4-layer, all FETs on top over a tight ground plane
Places all 160 footprints, sets the stackup and board outline, and lands
DRC-clean at 0 violations (382 unconnected is expected -- nothing routed).

The layer split is the whole point, and it is not the one I first
suggested. Loop inductance is set by distance to the RETURN PLANE, not by
how the FETs are stacked:

    high side top / low side bottom   1.60 mm  4.36 nH  13.1 V overshoot
    all FETs top, return on B.Cu      1.60 mm  4.36 nH  13.1 V
    all FETs top, In1 at 0.5 mm       0.50 mm  1.36 nH   4.1 V
    all FETs top, In1 at 0.2 mm       0.20 mm  0.54 nH   1.6 V   <- this

Splitting the half-bridge across the board is intuitively appealing and
about 8x worse, because it forces the return through the full board
thickness. So all twelve FETs sit on F.Cu with an unbroken PGND plane
0.2 mm beneath them, and the stackup is asymmetric on purpose. At 150 A
with 50 ns edges (3 A/ns) that is 14.2 V peak on a 40 V FET instead of
25.7 V.

Floorplan: current flows straight down each phase column -- DC+ pour, 24
ceramics directly above the high-side drains, HS pair, phase pour, LS
pair, shunt, PGND. FETs are rotated 90 so the source/gate edge faces down
and the drain paddle faces the pour above it; rotating them the other way
doubles the loop area. Three B.Cu lanes carry each phase to its own motor
terminal, and all logic is consolidated at x < 29 to keep those lanes
clear.

Resolves ESC-004: the placeholder terminal was a 2.5 sqmm wire pad (~25 A)
with a 25 mm strain-relief tail, unplaceable and badly underrated.
Replaced with a generated 3.6 mm / 9 mm dual-sided land pattern for 8 AWG.

Resolves ESC-013 (new): KiCad's _ThermalVias variant of the DRV8323R
footprint embeds 0.2 mm vias, below the 0.3 mm realistic minimum for 2 oz
copper. Switched to the plain land pattern; thermal vias go in by hand.

Three pcbnew quirks worth knowing, all of which cost a debugging round:
board.Remove() invalidat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
Parts:
- U201: footprint Package_DFN_QFN:Texas_RGZ0048A_VQFN-48-1EP_7x7mm_P0.5mm_EP5.15x5.15mm_ThermalVias -> Package_DFN_QFN:Texas_RGZ0048A_VQFN-48-1EP_7x7mm_P0.5mm_EP5.15x5.15mm
